Commit message: robot urdf -> commit
Signed-off-by: Ngochuy2137 <huy.nguyenngoc2137@gmail.com>

File: urdf/diff_robot.urdf (robot description, URDF)
Before this commit: robot nav2_mr_sim, 7 links, 6 joints
Links:
- removed link lidar_link
- added link base_scan, mass 0.114; collision cylinder length=0.05 radius=0.05; visual cylinder length=0.05 radius=0.1
- link base_link: geometry visual box size=0.35 0.2 0.1
- link caster_wheel: geometry collision sphere radius=0.025; visual sphere radius=0.025
- link left_wheel: geometry collision cylinder length=0.05 radius=0.05; visual cylinder length=0.05 radius=0.05
- link right_wheel: geometry collision cylinder length=0.05 radius=0.05; visual cylinder length=0.05 radius=0.05
Joints:
- joint base_lidar_joint: child lidar_link -> base_scan; origin xyz=0.0 0.0 0.225 rpy=0.0 0.0 0.0 -> xyz=0.0 0.0 0.15 rpy=0.0 0.0 0.0
- joint caster_wheel_joint: origin xyz=0.2 0.0 -0.05 rpy=0.0 0.0 0.0 -> xyz=0.125 0.0 0.0 rpy=0.0 0.0 0.0
- joint imu_joint: origin xyz=0.1 0.1 0.1 rpy=0.0 0.0 0.0 -> xyz=0.05 0.05 0.05 rpy=0.0 0.0 0.0
- joint left_wheel_joint: origin xyz=-0.175 0.225 0.0 rpy=0 0.0 0.0 -> xyz=-0.0875 0.125 0.025 rpy=0 0.0 0.0
- joint right_wheel_joint: origin xyz=-0.175 -0.225 0.0 rpy=0 0.0 0.0 -> xyz=-0.0875 -0.125 0.025 rpy=0 0.0 0.0
